File: HARDWARE/EAGLE/mapesynth_2pag.brd (EAGLE design)
At the start: 110.5 x 114.3 mm, 48 parts

Commit message: Add files via upload
Parts:
- R11: value 150 -> 68
Changed lines of the file:
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@@
 <setting verticaltext="up"/>
 </settings>
-<grid distance="50" unitdist="mil" unit="mil" style="dots" multiple="1" display="yes" altdistance="0.025" altunitdist="inch" altunit="inch"/>
+<grid distance="10" unitdist="mil" unit="mil" style="dots" multiple="1" display="yes" altdistance="0.025" altunitdist="inch" altunit="inch"/>
 <layers>
 <layer number="1" name="Top" color="4" fill="1" visible="yes" active="yes"/>
@@
 <attribute name="VALUE" x="13.589" y="46.5074" size="1.27" layer="21" ratio="10" rot="R90"/>
 </element>
-<element name="R11" library="resistor" package="0207/10" value="150" x="7.112" y="52.07" smashed="yes" rot="R90">
+<element name="R11" library="resistor" package="0207/10" value="68" x="7.112" y="52.07" smashed="yes" rot="R90">
 <attribute name="NAME" x="7.366" y="42.672" size="1.27" layer="21" ratio="10" rot="R90"/>
 <attribute name="VALUE" x="7.747" y="49.8094" size="1.27" layer="21" ratio="10" rot="R90"/>
@@
 <contactref element="R2" pad="1"/>
 <contactref element="R3" pad="1"/>
-<contactref element="U$5" pad="P$3"/>
 <wire x1="21.59" y1="73.406" x2="23.368" y2="73.406" width="0.4064" layer="16"/>
 <wire x1="23.368" y1="73.406" x2="25.146" y2="71.628" width="0.4064" layer="16"/>
 <wire x1="25.146" y1="71.628" x2="25.146" y2="66.802" width="0.4064" layer="16"/>
 <wire x1="25.146" y1="66.802" x2="25.146" y2="29.21" width="0.4064" layer="16"/>
-<wire x1="25.146" y1="29.21" x2="26.416" y2="27.94" width="0.4064" layer="16"/>
-<wire x1="26.416" y1="27.94" x2="27.94" y2="27.94" width="0.4064" layer="16"/>
 <wire x1="22.352" y1="67.056" x2="22.352" y2="64.008" width="0.4064" layer="16"/>
 <wire x1="22.352" y1="67.056" x2="24.892" y2="67.056" width="0.4064" layer="16"/>
 <wire x1="24.892" y1="67.056" x2="25.146" y2="66.802" width="0.4064" layer="16"/>
+<contactref element="U$5" pad="P$3"/>
+<wire x1="25.146" y1="29.21" x2="26.416" y2="27.94" width="0.4064" layer="16"/>
+<wire x1="26.416" y1="27.94" x2="27.94" y2="27.94" width="0.4064" layer="16"/>
 </signal>
 <signal name="VCC">
@@
 <wire x1="11.938" y1="-21.336" x2="16.256" y2="-21.336" width="0.8128" layer="1"/>
 <wire x1="16.256" y1="-21.336" x2="17.526" y2="-22.606" width="0.8128" layer="1"/>
-<polygon width="0.3048" layer="16" isolate="0.4064">
+<polygon width="0.3048" layer="16" pour="cutout" isolate="0.4064">
 <vertex x="-16.51" y="82.55"/>
 <vertex x="93.98" y="82.55"/>
@@
 <vertex x="-16.51" y="-31.75"/>
 </polygon>
-<polygon width="0.3048" layer="1" isolate="0.3048">
+<polygon width="0.3048" layer="1" pour="cutout" isolate="0.3048">
 <vertex x="-16.51" y="82.55"/>
 <vertex x="93.98" y="82.55"/>
@@
 <contactref element="R13" pad="1"/>
 <contactref element="R10" pad="1"/>
-<contactref element="U$5" pad="P$4"/>
 <wire x1="9.906" y1="43.688" x2="12.954" y2="43.688" width="0.4064" layer="16"/>
-<wire x1="27.94" y1="25.4" x2="27.178" y2="25.4" width="0.4064" layer="16"/>
 <wire x1="27.178" y1="25.4" x2="24.13" y2="28.448" width="0.4064" layer="16"/>
 <wire x1="24.13" y1="28.448" x2="24.13" y2="39.37" width="0.4064" layer="16"/>
 <wire x1="24.13" y1="39.37" x2="20.066" y2="43.688" width="0.4064" layer="16"/>
 <wire x1="20.066" y1="43.688" x2="12.954" y2="43.688" width="0.4064" layer="16"/>
+<contactref element="U$5" pad="P$4"/>
+<wire x1="27.178" y1="25.4" x2="27.94" y2="25.4" width="0.4064" layer="16"/>
 </signal>
 <signal name="N$12">
